Commit message: done solo movement for multi diff-drive robots

File: urdf/diffdrive_wheel_robot_disc_bumper.urdf (robot description, URDF)
Before this commit: robot diffdrive_wheel_robot_disc_bumper, 9 links, 8 joints
Links:
- link base_link: geometry collision cylinder length=0.06 radius=0.05; visual cylinder length=0.06 radius=0.05
- link wheel_left_link: geometry collision cylinder length=0.01 radius=0.02; visual cylinder length=0.01 radius=0.015
- link wheel_right_link: geometry collision cylinder length=0.01 radius=0.02; visual cylinder length=0.01 radius=0.02
Joints:
- joint bumper_joint: origin xyz=0 0 0.038 rpy=0 0 0 -> xyz=0 0 0.058 rpy=0 0 0
- joint heading_marker_joint: origin xyz=0.03 0 0.04 rpy=0 0 0 -> xyz=0.03 0 0.06 rpy=0 0 0
